File: starbie.kicad_sch (KiCad schematic)
At the start: 7 parts, among them J1 Conn_01x04_Pin, J2 Conn_01x08_Pin, SW1 SW_Push, SW2 SW_Push, U1 XIAO-ESP32-C3-SMD, U2 DHT11

Commit message: Addeded BOM fixed stuff and added decorations
Connections:
- net DHT11 DATA: now also U1.2 (D1)
- net GPIO3: now also SW2.1
- removed net GPIO1: SW2.1, U1.2 (D1)
Changed lines of the file:
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@@
 		)
 	)
-	(label "GPIO1"
+	(label "DHT11 DATA"
 		(at 124.46 50.8 180)
 		(effects
@@
 		)
 	)
-	(label "GPIO1"
+	(label "GPIO3"
 		(at 31.75 60.96 180)
 		(effects

Commit message: Added new Gerbers
Connections:
- net GND: now also U1.18 (GND)
- removed net X: J2.5 (Pin_5), J2.6 (Pin_6), J2.7 (Pin_7), J2.8 (Pin_8), U1.1 (D0), U1.10 (D9/BOOT), U1.7 (D6), U1.8 (D7), U1.9 (D8)
- no-connect marks 0 -> 17
Changed lines of the file:
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@@
 		)
+	)
+	(no_connect
+		(at 113.03 116.84)
+	)
+	(no_connect
+		(at 124.46 69.85)
+	)
+	(no_connect
+		(at 147.32 78.74)
+	)
+	(no_connect
+		(at 151.13 34.29)
+	)
+	(no_connect
+		(at 143.51 34.29)
+	)
+	(no_connect
+		(at 166.37 66.04)
+	)
+	(no_connect
+		(at 143.51 78.74)
+	)
+	(no_connect
+		(at 139.7 34.29)
+	)
+	(no_connect
+		(at 124.46 46.99)
+	)
+	(no_connect
+		(at 166.37 62.23)
+	)
+	(no_connect
+		(at 166.37 69.85)
+	)
+	(no_connect
+		(at 166.37 58.42)
+	)
+	(no_connect
+		(at 113.03 111.76)
+	)
+	(no_connect
+		(at 113.03 119.38)
+	)
+	(no_connect
+		(at 135.89 34.29)
+	)
+	(no_connect
+		(at 154.94 34.29)
+	)
+	(no_connect
+		(at 113.03 114.3)
 	)
 	(wire
@@
 	(wire
 		(pts
-			(xy 171.45 50.8) (xy 166.37 50.8)
+			(xy 147.32 17.78) (xy 147.32 34.29)
 		)
 		(stroke
@@
 	(wire
 		(pts
-			(xy 180.34 54.61) (xy 166.37 54.61)
+			(xy 171.45 50.8) (xy 166.37 50.8)
 		)
 		(stroke
@@
 	(wire
 		(pts
-			(xy 40.64 101.6) (xy 31.75 101.6)
+			(xy 180.34 54.61) (xy 166.37 54.61)
 		)
 		(stroke
@@
 	(wire
 		(pts
-			(xy 121.92 104.14) (xy 113.03 104.14)
+			(xy 40.64 101.6) (xy 31.75 101.6)
 		)
 		(stroke
@@
 	(wire
 		(pts
-			(xy 194.31 123.19) (xy 194.31 120.65)
+			(xy 121.92 104.14) (xy 113.03 104.14)
 		)
 		(stroke
@@
 	(wire
 		(pts
-			(xy 170.18 46.99) (xy 166.37 46.99)
+			(xy 194.31 123.19) (xy 194.31 120.65)
 		)
 		(stroke
@@
 	(wire
 		(pts
-			(xy 121.92 101.6) (xy 113.03 101.6)
+			(xy 143.51 20.32) (xy 143.51 17.78)
 		)
 		(stroke
@@
 	(wire
 		(pts
+			(xy 170.18 46.99) (xy 166.37 46.99)
+		)
+		(stroke
+			(width 0)
+			(type default)
+		)
+	)
+	(wire
+		(pts
+			(xy 121.92 101.6) (xy 113.03 101.6)
+		)
+		(stroke
+			(width 0)
+			(type default)
+		)
+	)
+	(wire
+		(pts
 			(xy 31.75 101.6) (xy 31.75 96.52)
+		)
+		(stroke
+			(width 0)
+			(type default)
+		)
+	)
+	(wire
+		(pts
+			(xy 143.51 17.78) (xy 147.32 17.78)
 		)
 		(stroke
@@
 		)
 	)
-	(label "X"
-		(at 113.03 114.3 0)
-		(effects
-			(font
-				(size 1.27 1.27)
-			)
-			(justify left bottom)
-		)
-	)
-	(label "x"
-		(at 166.37 59.69 180)
-		(effects
-			(font
-				(size 1.27 1.27)
-			)
-			(justify right bottom)
-		)
-	)
 	(label "GPIO2"
 		(at 124.46 54.61 180)
@@
 		)
 	)
-	(label "X"
-		(at 166.37 69.85 0)
-		(effects
-			(font
-				(size 1.27 1.27)
-			)
-			(justify left bottom)
-		)
-	)
 	(label "GPIO3"
 		(at 124.46 58.42 180)
@@
 		)
 	)
-	(label "X"
-		(at 113.03 119.38 0)
-		(effects
-			(font
-				(size 1.27 1.27)
-			)
-			(justify left bottom)
-		)
-	)
 	(label "GPIO3"
 		(at 31.75 60.96 180)
@@
 		)
 	)
-	(label "X"
-		(at 166.37 66.04 0)
-		(effects
-			(font
-				(size 1.27 1.27)
-			)
-			(justify left bottom)
-		)
-	)
-	(label "X"
-		(at 124.46 46.99 180)
-		(effects
-			(font
-				(size 1.27 1.27)
-			)
-			(justify right bottom)
-		)
-	)
 	(label "SCL"
 		(at 34.29 96.52 270)
@@
 		)
 	)
-	(label "X"
-		(at 124.46 69.85 180)
-		(effects
-			(font
-				(size 1.27 1.27)
-			)
-			(justify right bottom)
-		)
-	)
-	(label "X"
-		(at 113.03 116.84 0)
-		(effects
-			(font
-				(size 1.27 1.27)
-			)
-			(justify left bottom)
-		)
-	)
 	(label "SCL"
 		(at 124.46 62.23 180)
@@
 		)
 	)
-	(label "X"
-		(at 113.03 111.76 0)
-		(effects
-			(font
-				(size 1.27 1.27)
-			)
-			(justify left bottom)
-		)
-	)
 	(label "DHT11 DATA"
 		(at 194.31 123.19 180)
@@
 			)
 			(justify right bottom)
-		)
-	)
-	(label "X"
-		(at 166.37 62.23 0)
-		(effects
-			(font
-				(size 1.27 1.27)
-			)
-			(justify left bottom)
 		)
 	)
@@
 					(unit 1)
 				)
+			)
+		)
+	)
+	(symbol
+		(lib_id "power:GND")
+		(at 143.51 20.32 0)
+		(unit 1)
+		(body_style 1)
+		(exclude_from_sim no)
+		(in_bom yes)
+		(on_board yes)
+		(in_pos_files yes)
+		(dnp no)
+		(fields_autoplaced yes)
+		(property "Reference" "#PWR013"
+			(at 143.51 26.67 0)
+			(hide yes)
+			(show_name no)
+			(do_not_autoplace no)
+			(effects
+				(font
+					(size 1.27 1.27)
+				)
+			)
+		)
+		(property "Value" "GND"
+			(at 143.51 25.4 0)
+			(show_name no)
+			(do_not_autoplace no)
+			(effects
+				(font
+					(size 1.27 1.27)
+				)
+			)
+		)
+		(property "Footprint" ""
+			(at 143.51 20.32 0)
+			(hide yes)
+			(show_name no)
+			(do_not_autoplace no)
+			(effects
+				(font
+					(size 1.27 1.27)
+				)
+			)
+		)
+		(property "Datasheet" ""
+			(at 143.51 20.32 0)
+			(hide yes)
+			(show_name no)
+			(do_not_autoplace no)
+			(effects
+				(font
+					(size 1.27 1.27)
+				)
+			)
+		)
+		(property "Description" "Power symbol creates a global label with name \"GND\" , ground"
+			(at 143.51 20.32 0)
+			(hide yes)
+			(show_name no)
+			(do_not_autoplace no)
+			(effects
+				(font
+					(size 1.27 1.27)
+				)
+			)
+		)
+		(pin "1"
+		)
+		(instances
+			(project "starbie"
+				(path "/4e57b60e-1224-48f9-935a-2d2f539b6322"
+					(reference "#PWR013")
+					(unit 1)
+				)
